File: lm317-lm337-dual-rail-psu/Dual_Rail_Linear_PSU.kicad_pcb (KiCad board)
At the start: 2 copper layers, 75 x 50 mm, 20 parts, among them U1 LM317_TO-220, U2 LM337_TO220

Commit message: Finished Routing
Routing:
- net /-30V: track 0.00 -> 61.5 mm
- net /-12V: track 0.00 -> 54.4 mm
- net /12V: track 0.00 -> 50.7 mm
- net Net-(U2-ADJ): track 0.00 -> 47.4 mm
- net /30V: track 0.00 -> 46.7 mm
- net Net-(U1-ADJ): track 0.00 -> 23.5 mm
- net GND: track 0.00 -> 13.4 mm
- added copper zone on B.Cu, net GND
Other:
- outline, holes or cut-outs redrawn
