File: BipedRobot/BipedRobot.kicad_sch (KiCad schematic)
At the start: 17 parts, among them J2 Conn_01x02, U1 ESP32-DEVKIT-V1

Commit message: PCB done
Parts:
- removed GreenLED, RedLED: LED, symbol Device:LED
- removed J2: Conn_01x02, symbol Connector_Generic:Conn_01x02
- removed R1, R2: 330, symbol Device:R
- added C5, C7: 470uf, Capacitor_THT:CP_Radial_D10.0mm_P5.00mm, symbol Device:C
- added C6: 2200uF, Capacitor_THT:CP_Radial_D16.0mm_P7.50mm, symbol Device:C
- added H1, H2, H3, H4: MountingHole, MountingHole:MountingHole_3.2mm_M3, symbol Mechanical:MountingHole
- added LIPO_Batt1: Conn_01x02, Connector_AMASS:AMASS_XT30UPB-M_1x02_P5.0mm_Vertical, symbol Connector_Generic:Conn_01x02
- added LM2596Output1, Switch1: Conn_01x02, Connector_Wire:SolderWire-0.5sqmm_1x02_P4.6mm_D0.9mm_OD2.1mm, symbol Connector_Generic:Conn_01x02
- added TP3, TP4, TP5: TestPoint, TestPoint:TestPoint_Pad_D2.0mm, symbol Connector:TestPoint
- added UBEC_Input1, UBEC_Output1: Conn_01x02, Connector_Wire:SolderWire-1sqmm_1x02_P5.4mm_D1.4mm_OD2.7mm, symbol Connector_Generic:Conn_01x02
- C1, C2: value 0.1uf -> 100nf; footprint (none) -> Capacitor_THT:C_Disc_D5.0mm_W2.5mm_P5.00mm
- LM2596Input1: renamed from PowerSwitch; footprint (none) -> Connector_Wire:SolderWire-0.5sqmm_1x02_P4.6mm_D0.9mm_OD2.1mm
- LeftMotor1: renamed from LeftMotor; footprint (none) -> Connector_JST:JST_XH_B6B-XH-A_1x06_P2.50mm_Vertical
- LeftServo1, LeftServo2, RightServo1, RightServo2: footprint (none) -> Connector_PinHeader_2.54mm:PinHeader_1x03_P2.54mm_Vertical
- MPU6050: footprint OC09600:MODULE_OC09600 -> MPU6050:MODULE_OC09600
- RightMotor1: renamed from RightMotor; footprint (none) -> Connector_JST:JST_XH_B6B-XH-A_1x06_P2.50mm_Vertical
- TB6612FNG1: renamed from TB6612FNG; footprint ROB-14450:MODULE_ROB-14450 -> TB6612FNG:MODULE_ROB-14450
Connections:
- net +3V3 is gone; now on net 3V3: MPU6050.VCC, TB6612FNG1.2 (VCC), U1.1 (3V3)
- net 3V3: now also TP5.1
- net D13: now also TB6612FNG1.16 (PWMA); no longer TB6612FNG1.13 (STBY)
- net D14: now also TB6612FNG1.15 (AI2); no longer TB6612FNG1.10 (PWMB)
- net D25: now also TB6612FNG1.12 (BI1); no longer TB6612FNG1.16 (PWMA)
- net D26: now also TB6612FNG1.13 (STBY); no longer TB6612FNG1.14 (AI1)
- net D27: now also TB6612FNG1.14 (AI1); no longer TB6612FNG1.15 (AI2)
- net D32: now also TB6612FNG1.10 (PWMB); no longer TB6612FNG1.12 (BI1)
- net D34: now also RightMotor1.4 (Pin_4); no longer RightMotor1.3 (Pin_3)
- net D35: now also RightMotor1.3 (Pin_3); no longer RightMotor1.4 (Pin_4)
- net GND: now also LM2596Input1.2 (Pin_2), C5.2, C6.2, C7.2, LIPO_Batt1.2 (Pin_2), LM2596Output1.2 (Pin_2), UBEC_Input1.2 (Pin_2), UBEC_Output1.2 (Pin_2)
- net RX2: now also LeftServo1.3 (Pin_3), U1.6 (RX2); no longer LeftServo2.3 (Pin_3), U1.7 (TX2)
- net TX2: now also LeftServo2.3 (Pin_3), U1.7 (TX2); no longer LeftServo1.3 (Pin_3), U1.6 (RX2)
- net Switch+: now reaches TB6612FNG1.1 (VM)
- net Switch+: now also LM2596Input1.1 (Pin_1), C5.1, Switch1.2 (Pin_2), UBEC_Input1.1 (Pin_1)
- net LM2596_5V: now reaches U1.30 (VIN)
- net LM2596_5V: now also C7.1, LM2596Output1.1 (Pin_1), TP3.1
- net 6V renamed UBEC_OUT+
- net UBEC_OUT+: now also C6.1, TP4.1, UBEC_Output1.1 (Pin_1)
- net D12: no longer names the net of U1.27 (D12)
- net D15: no longer names the net of U1.3 (D15)
- net D2: no longer names the net of U1.4 (D2)
- net D23: no longer names the net of U1.15 (D23)
- net D4: no longer names the net of U1.5 (D4)
- net D5: no longer names the net of U1.8 (D5)
- new net BATT+: LIPO_Batt1.1 (Pin_1), Switch1.1 (Pin_1)
- no-connect marks 6 -> 12
Other:
- note added: "BuckConverter Terminals"
- note added: "DC Motor Terminals"
- note added: "ESP-32 Microcontroller"
- note added: "MPU6050"
- note added: "Motor Driver"
- note added: "Mounting Holes"
- note added: "Power"
- note added: "Servo Terminals"
- note added: "UBEC Terminals"
- moved on the sheet: C1, C2, LM2596Input1, LeftMotor1, LeftServo1, LeftServo2, MPU6050, RightMotor1, RightServo1, RightServo2, TB6612FNG1, U1
